File: Sensor-Firebeetle.kicad_sch (KiCad schematic)
At the start: 13 parts, among them J1 Solar Panel, J2 Battery, SW1 Sensor Number, U1 DFR0654, U2 BME280, U3 TP4056

Commit message: 3.3V for switches
Connections:
- net +3.3V: now also SW1.3, SW1.4
- net +5V: no longer SW1.3, SW1.4
Changed lines of the file:
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@@
     (effects (font (size 2.9972 2.9972) (thickness 0.5994) bold) (justify left bottom))
+  )
+  (global_label "+3.3V" (shape input) (at 93.98 53.34 270) (fields_autoplaced)
+    (effects (font (size 1.27 1.27)) (justify right))
+    (property "Intersheet References" "${INTERSHEET_REFS}" (id 0) (at 94.0594 61.349 90)
+      (effects (font (size 1.27 1.27)) (justify right) hide)
+    )
   )
   (global_label "GND" (shape input) (at 172.72 40.64 0) (fields_autoplaced)
@@
     )
   )
-  (global_label "+5V" (shape input) (at 93.98 53.34 270) (fields_autoplaced)
-    (effects (font (size 1.27 1.27)) (justify right))
-    (property "Intersheet References" "${INTERSHEET_REFS}" (id 0) (at 218.44 -148.59 0)
-      (effects (font (size 1.27 1.27)) hide)
-    )
-  )
