File: Sensor-D1Mini.kicad_sch (KiCad schematic)
At the start: 13 parts, among them J1 Solar Panel, J2 Battery, SW1 Sensor Number, U1 BME280, U2 mini_esp32, U4 TP4056

Commit message: 3.3V for switches
Connections:
- net +3.3V: now also SW1.3, SW1.4
- net +5V: no longer SW1.3, SW1.4
Changed lines of the file:
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@@
+    )
+  )
+  (global_label "+3.3V" (shape input) (at 113.03 62.23 270) (fields_autoplaced)
+    (effects (font (size 1.27 1.27)) (justify right))
+    (property "Intersheet References" "${INTERSHEET_REFS}" (id 0) (at 113.1094 70.239 90)
+      (effects (font (size 1.27 1.27)) (justify right) hide)
     )
   )
@@
       (effects (font (size 1.27 1.27)) hide)
     )
-  )
-  (global_label "+5V" (shape input) (at 113.03 62.23 270) (fields_autoplaced)
-    (effects (font (size 1.27 1.27)) (justify right))
-    (property "Intersheet References" "${INTERSHEET_REFS}" (id 0) (at 237.49 -139.7 0)
-      (effects (font (size 1.27 1.27)) hide)
-    )
